Commit message: rename motor joint

File: flypulator_description/urdf/multirotor_base.xacro (robot description, xacro)
@@ -68,5 +68,5 @@
   <xacro:macro name="vertical_rotor"
     params="robot_namespace suffix direction motor_constant moment_constant parent mass_rotor radius_rotor time_constant_up time_constant_down max_rot_velocity motor_number rotor_drag_coefficient rolling_moment_coefficient color use_own_mesh mesh *origin *inertia">
-    <joint name="motor_joint${motor_number}" type="continuous">
+    <joint name="motor_joint${motor_number+1}" type="continuous">
       <xacro:insert_block name="origin" />
       <axis xyz="0 0 1" />
