Commit message: correct orientation of the coordinate frames for blade and motor joints

File: flypulator_description/urdf/hexarotor_igs.urdf (robot description, URDF)
Before this commit: robot Hexacopter, 19 links, 18 joints
Links:
- link arm_link_1: mass 0.0825353339299331 -> 0.11307
- link arm_link_2: mass 0.082535 -> 0.113071616632983
- link arm_link_3: mass 0.082535 -> 0.113071616827671
- link arm_link_4: mass 0.082535 -> 0.113071614536244
- link arm_link_5: mass 0.0825353316162353 -> 0.113071612209128
- link arm_link_6: mass 0.082535 -> 0.11307
- link blade_link_2: mass 0.0627428767635787 -> 0.062743
- link blade_link_3: mass 0.0627473719638348 -> 0.062747
- link motor_link_1: mass 0.0980406960173389 -> 0.098041
- link motor_link_5: mass 0.098041 -> 0.0980407161578018
Joints:
- joint arm_joint_1: origin xyz=-1.7301E-05 -0.043794 0.03 rpy=1.3062E-16 2.419E-20 3.1412 -> xyz=0.037926 -0.021897 0.03 rpy=6.5556E-16 -1.0144E-15 -2.0944
- joint arm_joint_2: origin xyz=0.036818 -0.021277 0.03 rpy=1.4184E-15 1.159E-16 -2.0948 -> xyz=0.036827 0.021262 0.03 rpy=8.0241E-16 -8.459E-16 -1.0472
- joint arm_joint_3: origin xyz=0.037928 0.021878 0.03 rpy=1.2301E-15 4.3358E-14 -1.0476 -> xyz=0 0.043785 0.03 rpy=8.9162E-17 4.3411E-14 -1.1102E-16
- joint arm_joint_4: origin xyz=1.7302E-05 0.043795 0.03 rpy=-0.0005299 2.7433E-07 0.00064712 -> xyz=-0.0379272628526742 0.0218973154176168 0.03 rpy=-0.000529898657228908 2.74334852536435E-07 1.04823974425529
- joint arm_joint_5: origin xyz=-0.036818 0.021277 0.03 rpy=-3.7758E-16 -1.4672E-15 1.0468 -> xyz=-0.0368267925361943 -0.0212619585841622 0.0300000000000001 rpy=2.38424860458359E-16 -5.05424148413291E-16 2.09439510239319
- joint arm_joint_6: origin xyz=-0.037928 -0.021878 0.03 rpy=-2.0233E-16 2.2195E-16 2.094 -> xyz=0 -0.0437852352480966 0.0300000000000001 rpy=9.38614440953606E-16 1.69378355161205E-16 -3.14159265358979
- joint blade_joint_1: origin xyz=0 0.046 0 rpy=3.1416 -0.0021799 -3.1416 -> xyz=0 0.046 0 rpy=-2.1319E-15 0.0021799 -2.2359E-18
- joint blade_joint_2: origin xyz=0 0.046 0 rpy=3.1416 1.0573 3.1416 -> xyz=0 0.046 0 rpy=1.3878E-17 -5.5511E-17 -7.7716E-16
- joint blade_joint_3: origin xyz=0.010849 0.044702 0 rpy=-3.1416 -0.0017735 2.9035 -> xyz=0 0.046 0 rpy=-1.3878E-17 -1.1102E-16 4.1155E-08
- joint blade_joint_4: origin xyz=-0.010817 0.04471 0 rpy=-3.1416 -0.0021575 -2.9042 -> xyz=0 0.046 0 rpy=2.3091E-15 0.0021575 5.5511E-17
- joint blade_joint_5: origin xyz=0.010784 0.044718 0 rpy=6.1201E-15 0.0017735 -0.23665 -> xyz=0 0.046 0 rpy=-6.1062E-15 0.0017735 7.494E-16
- joint blade_joint_6: origin xyz=-0.010817 0.04471 0 rpy=-3.1416 -0.0017735 -2.9042 -> xyz=0 0.046 0 rpy=1.0131E-15 0.0017735 2.7756E-17
- joint motor_joint_1: origin xyz=0.0011025 0.5623 0.0048775 rpy=1.5704 0.23736 -0.0018246 -> xyz=0.0011025 0.5623 0.0048775 rpy=1.5712 -0.23736 3.1398
- joint motor_joint_2: origin xyz=-0.001249 0.56231 0.0048421 rpy=1.5712 -0.23736 -0.0018246 -> xyz=-0.001249 0.56231 0.0048421 rpy=1.5704 0.23736 3.1398
- joint motor_joint_3: origin xyz=0.0011025 0.56231 0.0048775 rpy=1.5704 -0.00072585 -0.0017235 -> xyz=0.0011025 0.56231 0.0048775 rpy=1.5708 -0.23736 -3.1416
- joint motor_joint_4: origin xyz=-0.00066294 0.5623 0.00514 rpy=1.5717 2.0749E-06 -0.0027659 -> xyz=-0.000662937524737199 0.56229546947751 0.00514004450059716 rpy=1.56982209369664 0.237363119054977 3.13859762470708
- joint motor_joint_5: origin xyz=0.0011025 0.56231 0.0048775 rpy=1.5704 0.00071878 -0.0017241 -> xyz=0.001102462209182 0.562306513541 0.00487752564526311 rpy=1.57122537643973 -0.237364397815691 3.13976801289026
- joint motor_joint_6: origin xyz=-0.001249 0.56231 0.0048421 rpy=1.5712 -1.6851E-16 -0.0017238 -> xyz=-0.00124895892184055 0.562306513541 0.00484208436052314 rpy=1.57036727715008 0.237364397815704 3.13976801289032

Commit message: change blade coordinate frame orientation to keep consistent with original aerodynamic model

File: flypulator_description/urdf/hexarotor_igs.urdf (robot description, URDF)
Before this commit: robot drone, 19 links, 18 joints
Links:
- link arm_link_4: mass 0.113071614536244 -> 0.113071614536243
- link blade_link_2: mass 0.062743 -> 0.0627428767604964
- link blade_link_3: mass 0.062747 -> 0.0627473719638348
- link blade_link_4: mass 0.062745 -> 0.062744669954973
Joints:
- joint arm_joint_1: origin xyz=0.037926 -0.021897 0.03 rpy=6.5556E-16 -1.0144E-15 -2.0944 -> xyz=0.0379263277638919 -0.0218967755438572 0.03 rpy=6.5556015652822E-16 -1.01435265127275E-15 -2.09439510239319
- joint arm_joint_2: origin xyz=0.036827 0.021262 0.03 rpy=8.0241E-16 -8.459E-16 -1.0472 -> xyz=0.0368267925361948 0.0212619585841613 0.0300000000000008 rpy=8.02409225127727E-16 -8.45899975464507E-16 -1.0471975511966
- joint arm_joint_3: origin xyz=0 0.043785 0.03 rpy=8.9162E-17 4.3411E-14 -1.1102E-16 -> xyz=0 0.0437852352480928 0.0300000000000009 rpy=8.9161997561106E-17 4.34108246398995E-14 -1.11022302462516E-16
- joint blade_joint_1: axis 0 1 0 -> 0 0 1; origin xyz=0 0.046 0 rpy=-2.1319E-15 0.0021799 -2.2359E-18 -> xyz=0 0 0.046 rpy=6.1162E-18 -8.1315E-20 0
- joint blade_joint_2: axis 0 1 0 -> 0 0 1; origin xyz=0 0.046 0 rpy=1.3878E-17 -5.5511E-17 -7.7716E-16 -> xyz=0 0 0.046 rpy=8.0491E-16 0 -5.5511E-17
- joint blade_joint_3: axis 0 1 0 -> 0 0 1; origin xyz=0 0.046 0 rpy=-1.3878E-17 -1.1102E-16 4.1155E-08 -> xyz=0 0 0.046 rpy=-4.1154E-08 2.7756E-17 -5.5511E-17
- joint blade_joint_4: axis 0 1 0 -> 0 0 1; origin xyz=0 0.046 0 rpy=2.3091E-15 0.0021575 5.5511E-17 -> xyz=0 0 0.046 rpy=-8.888E-17 -6.7763E-20 -4.3368E-19
- joint blade_joint_5: axis 0 1 0 -> 0 0 1; origin xyz=0 0.046 0 rpy=-6.1062E-15 0.0017735 7.494E-16 -> xyz=0 0 0.046 rpy=-7.7716E-16 0 0
- joint blade_joint_6: axis 0 1 0 -> 0 0 1; origin xyz=0 0.046 0 rpy=1.0131E-15 0.0017735 2.7756E-17 -> xyz=0 0 0.046 rpy=-1.1102E-16 1.3878E-17 -5.5511E-17
- joint motor_joint_1: origin xyz=0.0011025 0.5623 0.0048775 rpy=1.5712 -0.23736 3.1398 -> xyz=0.0011025 0.5623 0.0048775 rpy=-0.23736 -0.00041702 -1.5725
- joint motor_joint_2: origin xyz=-0.001249 0.56231 0.0048421 rpy=1.5704 0.23736 3.1398 -> xyz=-0.00124895892184227 0.562306513541 0.00484208436052164 rpy=0.237364418851718 0.000417019559747398 -1.57252008000707
- joint motor_joint_3: origin xyz=0.0011025 0.56231 0.0048775 rpy=1.5708 -0.23736 -3.1416 -> xyz=0.00110246220918394 0.562306513541 0.00487752564526059 rpy=-0.237364418851689 -0.000417019559749972 -1.57252008000707
- joint motor_joint_4: origin xyz=-0.000662937524737199 0.56229546947751 0.00514004450059716 rpy=1.56982209369664 0.237363119054977 3.13859762470708 -> xyz=-0.000662937524737199 0.56229546947751 0.00514004450059716 rpy=0.237363227515671 0.000946916948792575 -1.5735622739509
- joint motor_joint_5: origin xyz=0.001102462209182 0.562306513541 0.00487752564526311 rpy=1.57122537643973 -0.237364397815691 3.13976801289026 -> xyz=0.001102462209182 0.562306513541 0.00487752564526311 rpy=-0.237364418851719 -0.000417019559769994 -1.57252008000713
- joint motor_joint_6: origin xyz=-0.00124895892184055 0.562306513541 0.00484208436052314 rpy=1.57036727715008 0.237364397815704 3.13976801289032 -> xyz=-0.00124895892184055 0.562306513541 0.00484208436052314 rpy=0.237364418851732 0.000417019559751141 -1.57252008000707

Commit message: correct motors and propellers orientation, add dummy root link without inertial info. for gazebo

File: flypulator_description/urdf/hexarotor_igs.urdf (robot description, URDF)
Before this commit: robot drone, 19 links, 18 joints
Links:
- added link dummy_link, mass 0; collision mesh filename=package://flypulator_description/meshes/dummy_link.STL; visual mesh filename=package://flypulator_description/meshes/dummy_link.STL
- added link foot_link_left, mass 0.63218; collision mesh filename=package://flypulator_description/meshes/foot_link_left.STL; visual mesh filename=package://flypulator_description/meshes/foot_link_left.STL
- added link foot_link_right, mass 0.63218; collision mesh filename=package://flypulator_description/meshes/foot_link_right.STL; visual mesh filename=package://flypulator_description/meshes/foot_link_right.STL
- link arm_link_2: mass 0.113071616632983 -> 0.11307
- link arm_link_3: mass 0.113071616827671 -> 0.11307
- link arm_link_4: mass 0.113071614536243 -> 0.11307
- link arm_link_5: mass 0.113071612209128 -> 0.11307
- link base_link: mass 4.5104 -> 3.2461
- link blade_link_2: mass 0.0627428767604964 -> 0.062743
- link blade_link_3: mass 0.0627473719638348 -> 0.062747
- link blade_link_5: mass 0.062743 -> 0.0627428768132032
- link motor_link_2: mass 0.0980407364233949 -> 0.098041
- link motor_link_3: mass 0.0980407398276978 -> 0.098041
Joints:
- added joint base_joint: type fixed, parent dummy_link, child base_link, origin xyz=0 0 0 rpy=0 0 0, axis 0 0 0
- added joint foot_joint_right: type fixed, parent base_link, child foot_link_right, origin xyz=0.00062258 -0.40242 -0.1931 rpy=1.5708 1.0405 1.5708, axis 0 0 0
- added joint foot_link_left: type fixed, parent base_link, child foot_link_left, origin xyz=-0.00062258 0.40242 -0.1931 rpy=1.5708 1.0405 -1.5708, axis 0 0 0
- joint arm_joint_1: origin xyz=0.0379263277638919 -0.0218967755438572 0.03 rpy=6.5556015652822E-16 -1.01435265127275E-15 -2.09439510239319 -> xyz=0.037926 -0.021897 0.03 rpy=0 0 -2.0944
- joint arm_joint_2: origin xyz=0.0368267925361948 0.0212619585841613 0.0300000000000008 rpy=8.02409225127727E-16 -8.45899975464507E-16 -1.0471975511966 -> xyz=0.036827 0.021262 0.03 rpy=0 0 -1.0472
- joint arm_joint_3: origin xyz=0 0.0437852352480928 0.0300000000000009 rpy=8.9161997561106E-17 4.34108246398995E-14 -1.11022302462516E-16 -> xyz=0 0.043785 0.03 rpy=0 0 0
- joint arm_joint_4: origin xyz=-0.0379272628526742 0.0218973154176168 0.03 rpy=-0.000529898657228908 2.74334852536435E-07 1.04823974425529 -> xyz=-0.037927 0.021897 0.03 rpy=-0.0005299 2.7433E-07 1.0482
- joint arm_joint_5: origin xyz=-0.0368267925361943 -0.0212619585841622 0.0300000000000001 rpy=2.38424860458359E-16 -5.05424148413291E-16 2.09439510239319 -> xyz=-0.036827 -0.021262 0.03 rpy=0 0 2.0944
- joint arm_joint_6: origin xyz=0 -0.0437852352480966 0.0300000000000001 rpy=9.38614440953606E-16 1.69378355161205E-16 -3.14159265358979 -> xyz=0 -0.043785 0.03 rpy=9.3861E-16 1.6938E-16 -3.1416
- joint blade_joint_1: origin xyz=0 0 0.046 rpy=6.1162E-18 -8.1315E-20 0 -> xyz=0 0 0.046 rpy=0 0 0
- joint blade_joint_2: origin xyz=0 0 0.046 rpy=8.0491E-16 0 -5.5511E-17 -> xyz=0 0 0.046 rpy=0 0 0
- joint blade_joint_3: origin xyz=0 0 0.046 rpy=-4.1154E-08 2.7756E-17 -5.5511E-17 -> xyz=0 0 0.046 rpy=0 0 0
- joint blade_joint_4: origin xyz=0 0 0.046 rpy=-8.888E-17 -6.7763E-20 -4.3368E-19 -> xyz=0 0 0.046 rpy=0 0 0
- joint blade_joint_5: origin xyz=0 0 0.046 rpy=-7.7716E-16 0 0 -> xyz=0 0 0.046 rpy=0 0 0
- joint blade_joint_6: origin xyz=0 0 0.046 rpy=-1.1102E-16 1.3878E-17 -5.5511E-17 -> xyz=0 0 0.046 rpy=0 0 0
- joint motor_joint_2: origin xyz=-0.00124895892184227 0.562306513541 0.00484208436052164 rpy=0.237364418851718 0.000417019559747398 -1.57252008000707 -> xyz=-0.001249 0.56231 0.0048421 rpy=0.23736 0.00041702 -1.5725

Commit message: remove dummy_link temporary, which may causes error.

File: flypulator_description/urdf/hexarotor_igs.urdf (robot description, URDF)
Before this commit: robot drone, 22 links, 21 joints
Links:
- removed link dummy_link
Joints:
- removed joint base_joint
